File: veloR/veloR.kicad_pcb (KiCad board)
At the start: 2 copper layers, 120 x 89.6 mm, 44 parts, among them J3 DISPLAY, J4 Conn_01x10, J6 Cable_PAD, J9 Programador, M1 M1, M2 M2, SW1 SW_DPST_x2, SW10 SW_Push, U3 AMS1117-3.3, U6 ESP32-WROOM-32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

Commit message: Add files via upload
Parts:
- moved H2 2.66 mm to (163.8, 137.8)
- moved H1 2.57 mm to (125.7, 137.8)
- moved C14 2.39 mm to (158.7, 101.5)
- moved C2 2.39 mm to (130.6, 101.5)
- moved J4 1.75 mm to (156.2, 138.5)
Connections:
- net Net-(M1-Pin_1) renamed M4
- net Net-(M1-Pin_2) renamed M3
- net Net-(M2-Pin_1) renamed M2
- net Net-(M2-Pin_2) renamed M1
Routing:
- net M2: track 15.2 -> 0.00 mm
- net M1: track 15.2 -> 0.00 mm
- net M3: track 15.2 -> 0.00 mm
- net M4: track 15.1 -> 0.00 mm
- net GND: track 10.2 -> 0.00 mm
- net VCC: track 82.8 -> 86.5 mm
- net D2: track 11.4 -> 9.39 mm
- net D1: track 12.6 -> 11.0 mm
- net D3: track 10.3 -> 8.79 mm
- net D4: track 9.29 -> 8.26 mm
- net D5: track 8.74 -> 7.92 mm
- added copper zone on F.Cu, net M1
- added copper zone on F.Cu, net M2
- added copper zone on F.Cu, net M3
- added copper zone on F.Cu, net M4
Other:
- outline, holes or cut-outs redrawn

Commit message: Add files via upload
MODIFIQUE PANTALLA,  ACOMODE COSAS, ETC
Parts:
- added D1: D, Diode_SMD:D_SMA, F.Cu at (168.2, 111.3)
- added G***: LOGO, LOGO, F.Cu at (176.9, 127.1)
- added R5: 10k, Resistor_SMD:R_1206_3216Metric_Pad1.30x1.75mm_HandSolder, F.Cu at (182.6, 118.1)
- added R8: 10k, Resistor_SMD:R_1206_3216Metric_Pad1.30x1.75mm_HandSolder, F.Cu at (185.1, 118.1)
- moved C7 2.64 mm to (123.2, 119.6)
- moved C8 2.64 mm to (123.2, 121.8)
- moved C11 1.72 mm to (123.2, 108.2)
- moved C12 1.72 mm to (123.2, 106.0)
Connections:
- J4 pad 1: +5V -> 3V3
- J9 pad 3: +5V -> Net-(D1-A)
- U6 pad 27: unconnected-(U6-IO17-Pad27) -> INA2
- U6 pad 34: INA2 -> unconnected-(U6-IO5-Pad34)
Routing:
- net +5V: track 142.3 -> 82.5 mm, vias 2 -> 25
- net 3V3: track 130.7 -> 163.6 mm, vias 4 -> 26
- net SCL: track 57.2 -> 67.6 mm
- net Net-(D1-A): track 0.00 -> 4.95 mm
- net SDA: track 47.0 -> 51.2 mm
- net SW3: track 54.7 -> 56.8 mm
- net VCC: track 86.5 -> 85.6 mm
- net INA2: track 12.4 -> 13.1 mm
- added copper zone on B.Cu, net +5V
- added copper zone on F.Cu, net +5V
- added copper zone on B.Cu, net 3V3
- added copper zone on F.Cu, net 3V3
Other:
- board size 120 x 89.6 mm -> 120 x 88.5 mm

Commit message: Add files via upload
Parts:
- removed J6 (x2): Cable_PAD, MacroLib:Pololu_Micro_Bracket_Wheel_42mm
- added M3: Motor_DC, NUEVAS HUELLAS TREJO:motor 3600rpm, F.Cu at (123.3, 68.0)
- added M4: Motor_DC, NUEVAS HUELLAS TREJO:motor 3600rpm, F.Cu at (165.2, 72.1)
- C1, C13: footprint Capacitor_SMD:C_Elec_4x5.4 -> Capacitor_SMD:C_Elec_10x10.2
- J4: footprint Connector_PinHeader_2.54mm:PinHeader_1x10_P2.54mm_Horizontal -> Connector_JST:JST_XH_S10B-XH-A-1_1x10_P2.50mm_Horizontal
- moved J4 22.6 mm to (133.6, 138.5), turned to 0 degrees
- moved Alimentacion1 8.81 mm to (117.5, 90.5), turned to -90 degrees
- moved SW1 7.51 mm to (110.0, 95.0), turned to 0 degrees
- moved C1 4.21 mm to (127.0, 93.6), turned to -90 degrees
- moved C13 4.05 mm to (162.5, 93.6), turned to -90 degrees
- moved R1 0.87 mm to (109.8, 90.6), turned to 0 degrees
- moved D2 0.82 mm to (109.8, 87.4), turned to 0 degrees
- moved C5 0.32 mm to (131.1, 132.9)
Connections:
- J4 pad 1: 3V3 -> GND
- J4 pad 10: GND -> 3V3
- J4 pad 2: D8 -> D1
- J4 pad 3: D7 -> D2
- J4 pad 4: D6 -> D3
- J4 pad 5: D5 -> D4
- J4 pad 6: D4 -> D5
- J4 pad 7: D3 -> D6
- J4 pad 8: D2 -> D7
- J4 pad 9: D1 -> D8
Routing:
- net +5V: track 82.5 -> 94.9 mm, vias 25 -> 26
- net 3V3: track 163.6 -> 171.5 mm, vias 26 -> 27
- net VCC: track 85.6 -> 81.7 mm
- net VCC1: track 47.1 -> 50.1 mm
- net SW3: track 56.8 -> 58.8 mm
- net SDA: track 51.2 -> 52.7 mm
- added copper zone on B.Cu, net GND
Other:
- board size 120 x 88.5 mm -> 120.1 x 88.5 mm
